File: dram/dram.kicad_pcb (KiCad board)
At the start: 2 copper layers, 101.6 x 76.2 mm, 35 parts, among them J1 Raspberry_Pi_2_3, J2 Barrel_Jack_MountingPin, J4 Conn_01x04_Pin, Q1 DMG2305UX-13 MOSFET, Q10 2N7002, Q11 2N7002, Q12 2N7002, Q13 2N7002, Q14 2N7002, Q2 DMMT5401 PNP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

Commit message: Add files via upload
Parts:
- removed C2, C3, C4: 47n, Capacitor_SMD:C_1206_3216Metric_Pad1.33x1.80mm_HandSolder
- removed D3, D4, D5: LED, LED_SMD:LED_1206_3216Metric_Pad1.42x1.75mm_HandSolder
- removed Q10, Q11, Q12, Q4, Q5, Q6, Q7, Q8, Q9: 2N7002, Package_TO_SOT_SMD:SOT-23
- removed R5, R6, R7: 150, Resistor_SMD:R_1206_3216Metric_Pad1.30x1.75mm_HandSolder
- added C1: 47n, Capacitor_SMD:C_1206_3216Metric_Pad1.33x1.80mm_HandSolder, F.Cu at (92.1, 51.2)
- added C1: 47n, Capacitor_SMD:C_1206_3216Metric_Pad1.33x1.80mm_HandSolder, F.Cu at (73.9, 51.2)
- added C1: 47n, Capacitor_SMD:C_1206_3216Metric_Pad1.33x1.80mm_HandSolder, F.Cu at (92.1, 36.5)
- added D2: LED, LED_SMD:LED_1206_3216Metric_Pad1.42x1.75mm_HandSolder, F.Cu at (86.3, 32.8)
- added D2: LED, LED_SMD:LED_1206_3216Metric_Pad1.42x1.75mm_HandSolder, F.Cu at (68.2, 47.5)
- added D2: LED, LED_SMD:LED_1206_3216Metric_Pad1.42x1.75mm_HandSolder, F.Cu at (86.3, 47.5)
- added Q13: 2N7002, Package_TO_SOT_SMD:SOT-23, F.Cu at (68.2, 55.0)
- added Q13: 2N7002, Package_TO_SOT_SMD:SOT-23, F.Cu at (86.3, 40.3)
- added Q13: 2N7002, Package_TO_SOT_SMD:SOT-23, F.Cu at (86.3, 55.0)
- added Q14: 2N7002, Package_TO_SOT_SMD:SOT-23, F.Cu at (92.1, 40.3)
- added Q14: 2N7002, Package_TO_SOT_SMD:SOT-23, F.Cu at (92.1, 55.0)
- added Q14: 2N7002, Package_TO_SOT_SMD:SOT-23, F.Cu at (73.9, 55.0)
- added Q3: 2N7002, Package_TO_SOT_SMD:SOT-23, F.Cu at (92.1, 32.7)
- added Q3: 2N7002, Package_TO_SOT_SMD:SOT-23, F.Cu at (92.1, 47.4)
- added Q3: 2N7002, Package_TO_SOT_SMD:SOT-23, F.Cu at (73.9, 47.4)
- added R4: 150, Resistor_SMD:R_1206_3216Metric_Pad1.30x1.75mm_HandSolder, F.Cu at (86.3, 36.5)
- added R4: 150, Resistor_SMD:R_1206_3216Metric_Pad1.30x1.75mm_HandSolder, F.Cu at (68.2, 51.2)
- added R4: 150, Resistor_SMD:R_1206_3216Metric_Pad1.30x1.75mm_HandSolder, F.Cu at (86.3, 51.2)
- moved Q14 27.1 mm to (73.9, 40.3)
- moved Q3 26.3 mm to (73.9, 32.7)
- moved C1 26.1 mm to (73.9, 36.5)
- moved Q13 24.7 mm to (68.2, 40.3)
- moved R4 24.2 mm to (68.2, 36.5)
- moved D2 24.2 mm to (68.2, 32.8), turned to 180 degrees
- moved J2 22.9 mm to (27.5, 47.0), turned to 180 degrees
- moved D1 22.6 mm to (48.9, 38.7), turned to -90 degrees
- moved U1 21.7 mm to (43.2, 54.6), turned to -90 degrees
- moved J1 21.6 mm to (55.2, 27.3)
- moved Q1 19.2 mm to (48.3, 33.0), turned to 90 degrees
- moved Q2 18.7 mm to (45.1, 27.9), turned to -90 degrees
- moved R3 17.1 mm to (45.1, 38.7)
- moved J4 16.2 mm to (46.7, 43.8), turned to -90 degrees
- moved R1 15.8 mm to (48.3, 27.9), turned to -90 degrees
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Connections:
- J1 pad 15: /B0 -> unconnected-(J1-GPIO22-Pad15)
- J1 pad 16: /B1 -> unconnected-(J1-GPIO23-Pad16)
- J1 pad 18: /W0 -> unconnected-(J1-GPIO24-Pad18)
- J1 pad 21: unconnected-(J1-MISO0/GPIO9-Pad21) -> /B0
- J1 pad 22: /W1 -> unconnected-(J1-GPIO25-Pad22)
- J1 pad 23: unconnected-(J1-SCLK0/GPIO11-Pad23) -> /B1
- J1 pad 27: unconnected-(J1-ID_SD/GPIO0-Pad27) -> /W0
- J1 pad 29: unconnected-(J1-GCLK1/GPIO5-Pad29) -> /W1
Routing:
- net GND: track 16.2 -> 214.3 mm, vias 0 -> 2
- net +5V: track 8.70 -> 147.6 mm, vias 0 -> 4
- net /B1: track 0.00 -> 72.4 mm, vias 0 -> 2
- net /W1: track 0.00 -> 59.4 mm
- net /W0: track 8.09 -> 58.1 mm, vias 0 -> 1
- net /ZVD_OUT: track 0.00 -> 36.9 mm
- net /B0: track 17.6 -> 39.8 mm, vias 0 -> 2
- net +9V: track 0.00 -> 21.9 mm
- net +3V3: track 0.00 -> 21.6 mm
- net Net-(J2-Pad1): track 0.00 -> 18.6 mm
- net Net-(Q14-D): track 12.0 -> 28.8 mm
- net Net-(Q13-S): track 8.09 -> 22.9 mm
- net Net-(D2-A): track 5.72 -> 20.0 mm
- net Net-(D1-K): track 0.00 -> 10.1 mm
- net Net-(Q2-Pad1): track 0.00 -> 9.98 mm
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