File: dram/dram.kicad_sch (KiCad schematic)
At the start: 35 parts, among them J1 Raspberry_Pi_2_3, J2 Barrel_Jack_MountingPin, J4 Conn_01x04_Pin, Q1 DMG2305UX-13 MOSFET, Q10 2N7002, Q11 2N7002, Q12 2N7002, Q13 2N7002, Q14 2N7002, Q2 DMMT5401 PNP, Q3 2N7002, Q4 2N7002, Q5 2N7002, Q6 2N7002, Q7 2N7002, Q8 2N7002, Q9 2N7002

Commit message: Add files via upload
Parts:
- added C10, C11, C12, C13, C14, C15, C16, C5, C6, C7, C8, C9: 47n, Capacitor_SMD:C_1206_3216Metric_Pad1.33x1.80mm_HandSolder, symbol Device:C
- added D10, D11, D12, D13, D14, D15, D16, D17, D6, D7, D8, D9: LED, LED_SMD:LED_1206_3216Metric_Pad1.42x1.75mm_HandSolder, symbol Device:LED
- added Q15, Q16, Q17, Q18, Q19, Q20, Q21, Q22, Q23, Q24, Q25, Q26, Q27, Q28, Q29, Q30, Q31, Q32, Q33, Q34, Q35, Q36, Q37, Q38, Q39, Q40, Q41, Q42, Q43, Q44, Q45, Q46, Q47, Q48, Q49, Q50: 2N7002, Package_TO_SOT_SMD:SOT-23, symbol Transistor_FET:2N7002
- added R10, R11, R12, R13, R14, R15, R16, R17, R18, R19, R8, R9: 150, Resistor_SMD:R_1206_3216Metric_Pad1.30x1.75mm_HandSolder, symbol Device:R_US
Connections:
- net +5V: now also C10.1, C11.1, C12.1, C13.1, C14.1, C15.1, C16.1, C5.1, C6.1, C7.1, C8.1, C9.1, R10.1, R11.1, R12.1, R13.1, R14.1, R15.1, R16.1, R17.1, R18.1, R19.1, R8.1, R9.1
- net B0: now also J1.21 (MISO0/GPIO9), Q15.3 (D), Q39.3 (D); no longer J1.15 (GPIO22)
- net B1: now also J1.23 (SCLK0/GPIO11), Q18.3 (D), Q42.3 (D); no longer J1.16 (GPIO23)
- net GND: now also Q17.2 (S), Q20.2 (S), Q27.2 (S), Q28.2 (S), Q29.2 (S), Q36.2 (S), Q37.2 (S), Q38.2 (S), Q41.2 (S), Q44.2 (S), Q47.2 (S), Q50.2 (S)
- net W0: now also J1.27 (ID_SD/GPIO0), Q21.1 (G), Q24.1 (G), Q30.1 (G), Q33.1 (G); no longer J1.18 (GPIO24)
- net W1: now also J1.29 (GCLK1/GPIO5), Q22.1 (G), Q25.1 (G), Q31.1 (G), Q34.1 (G); no longer J1.22 (GPIO25)
- new net: D15.1 (K), Q44.3 (D)
- new net: D15.2 (A), R17.2
- new net: Q15.1 (G), Q16.1 (G), Q18.1 (G), Q19.1 (G), Q23.1 (G), Q26.1 (G), Q32.1 (G), Q35.1 (G)
- new net: Q23.2 (S), Q26.2 (S)
- new net: C9.2, Q26.3 (D), Q29.1 (G)
- new net: C15.2, Q46.3 (D), Q47.1 (G)
- new net: D16.1 (K), Q47.3 (D)
- new net: Q31.2 (S), Q34.2 (S)
- new net: C11.2, Q34.3 (D), Q36.1 (G)
- new net: D9.2 (A), R11.2
- new net: D13.2 (A), R15.2
- new net: Q39.1 (G), Q40.1 (G), Q42.1 (G), Q43.1 (G), Q45.1 (G), Q46.1 (G), Q48.1 (G), Q49.1 (G)
- new net: Q45.2 (S), Q46.2 (S)
- new net: Q22.2 (S), Q25.2 (S)
- new net: C8.2, Q25.3 (D), Q28.1 (G)
- new net: D6.1 (K), Q17.3 (D)
- new net: D6.2 (A), R8.2
- new net: D17.2 (A), R19.2
- new net: C5.2, Q16.3 (D), Q17.1 (G)
- new net: D14.1 (K), Q41.3 (D)
- new net: D14.2 (A), R16.2
- new net: D16.2 (A), R18.2
- new net: D12.2 (A), R14.2
- new net: C6.2, Q19.3 (D), Q20.1 (G)
- new net: C16.2, Q49.3 (D), Q50.1 (G)
- new net: D17.1 (K), Q50.3 (D)
- new net: D13.1 (K), Q38.3 (D)
- new net: Q42.2 (S), Q43.2 (S)
- new net: Q30.2 (S), Q33.2 (S)
- new net: C10.2, Q33.3 (D), Q38.1 (G)
- new net: Q39.2 (S), Q40.2 (S)
- new net: C13.2, Q40.3 (D), Q41.1 (G)
- new net: C14.2, Q43.3 (D), Q44.1 (G)
- new net: D10.1 (K), Q29.3 (D)
- new net: D10.2 (A), R12.2
- new net: Q48.2 (S), Q49.2 (S)
- new net: Q32.2 (S), Q35.2 (S)
- new net: D11.2 (A), R13.2
- new net: D9.1 (K), Q28.3 (D)
- new net: D8.1 (K), Q27.3 (D)
- new net: D8.2 (A), R10.2
- new net: Q15.2 (S), Q16.2 (S)
- new net: Q18.2 (S), Q19.2 (S)
- new net: Q21.2 (S), Q24.2 (S)
- new net: C7.2, Q24.3 (D), Q27.1 (G)
- new net: D7.1 (K), Q20.3 (D)
- new net: D7.2 (A), R9.2
- new net: D12.1 (K), Q37.3 (D)
- new net: C12.2, Q35.3 (D), Q37.1 (G)
- new net: D11.1 (K), Q36.3 (D)
- new net B2: Q21.3 (D), Q22.3 (D), Q23.3 (D), Q45.3 (D)
- new net B3: Q30.3 (D), Q31.3 (D), Q32.3 (D), Q48.3 (D)
Other:
- moved on the sheet: C1, C2, C3, C4, D1, D2, D3, D4, D5, J1, J2, J4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
